File: ataconso/ataconso-rev-a/ataconso-rev-a.kicad_sch (KiCad schematic)
At the start: 0 parts

Commit message: agregar primeras conexiones
Parts:
- added C1: 100n, symbol Device:C
- added C2: 10u, symbol Device:C_Polarized
- added R1: 10k, symbol Device:R
- added U1, U2: NE555D, Package_SO:SOIC-8_3.9x4.9mm_P1.27mm, symbol Timer:NE555D
Connections:
- new net: U1.3 (OUT), U2.2 (TRIG)
- new net: U2.6 (THRES), U2.7 (DISCH)
- new net: R1.2, U1.7 (DISCH)
- new net: C1.1, U1.5 (CONT)
- new net: C2.1, U1.2 (TRIG), U1.6 (THRES)
- new net GND: C1.2, C2.2, U1.1 (GND), U2.1 (GND)
- new net VCC: R1.1, U1.4 (~{RST}), U1.8 (VCC), U2.4 (~{RST}), U2.8 (VCC)
Other:
- note added: "555 derecha 1: a tierra 2: 3: 4: a Vcc 5: 6: 7: a 6 8: a Vcc"
- note added: "555 izquierda 1: a tierra 2: a tierra por capacitor 3: a 2 de 555 derecha 4: a Vcc 5: 6: a 2 7: 8: a Vcc"
- company: (none) -> piruetas SpA

Commit message: agreagr ataconso sch
Parts:
- added C3, C4: 100n, symbol Device:C
- added C5: C_Polarized, symbol Device:C_Polarized
- added J1: Screw_Terminal_01x02, symbol Connector:Screw_Terminal_01x02
- added R2: 1k, symbol Device:R
- added RV1, RV2: 100k, symbol Device:R_Potentiometer
- R1: value 10k -> 1k
Connections:
- net GND: now also C3.2, C4.2, J1.2 (Pin_2)
- net VCC: now also RV2.2
- net at U2.3 (OUT): now also C5.1
- net at U2.5 (CONT): now also C3.1
- net at U2.6 (THRES), U2.7 (DISCH): now also C4.1, R2.2
- net at R1.2, U1.7 (DISCH): now also RV1.2
- net at C2.1, U1.2 (TRIG), U1.6 (THRES): now also RV1.3
- new net: R2.1, RV2.3
- new net: C5.2, J1.1 (Pin_1)
- no-connect marks 0 -> 2
Other:
- note added: "555 derecha 1: a tierra 2: a 3 de 555 izq 3: 4: a Vcc 5: a tierra por C 100n 6: a tierra por C 100n 7: a 6, a tierra por C, a Vcc por R 8: a Vcc"
- note added: "555 izquierda 1: a tierra 2: a tierra por C 3: a 2 de 555 derecha 4: a Vcc 5: a tierra por C 100n 6: a 2 7: a Vcc por R 10k, a 2 por RV de 100k 8: a Vcc"
- note removed: "555 derecha 1: a tierra 2: 3: 4: a Vcc 5: 6: 7: a 6 8: a Vcc"
- note removed: "555 izquierda 1: a tierra 2: a tierra por capacitor 3: a 2 de 555 derecha 4: a Vcc 5: 6: a 2 7: 8: a Vcc"

Commit message: agregar nuevos C
Parts:
- removed C2: 10u, symbol Device:C_Polarized
- added C1: 10n, symbol Device:C
- renumbered C1 to C2, C4 to C3, C3 to C4
Connections:
- net GND: now also C1.2
- net at RV1.3, U1.2 (TRIG), U1.6 (THRES): now also C1.1
Changed lines of the file:
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@@
 		(dnp no)
 		(fields_autoplaced yes)
-		(property "Reference" "#PWR01"
+		(property "Reference" "#PWR05"
 			(at 58.42 83.82 0)
 			(hide yes)
@@
 			(project "ataconso-rev-a"
 				(path "/837c7b7b-d540-4609-998f-42c63488299f"
-					(reference "#PWR01")
+					(reference "#PWR05")
 					(unit 1)
 				)
@@
 		(dnp no)
 		(fields_autoplaced yes)
-		(property "Reference" "#PWR08"
+		(property "Reference" "#PWR02"
 			(at 33.02 83.82 0)
 			(hide yes)
@@
 			(project "ataconso-rev-a"
 				(path "/837c7b7b-d540-4609-998f-42c63488299f"
-					(reference "#PWR08")
+					(reference "#PWR02")
 					(unit 1)
 				)
@@
 		(dnp no)
 		(fields_autoplaced yes)
-		(property "Reference" "#PWR04"
+		(property "Reference" "#PWR09"
 			(at 96.52 49.53 0)
 			(hide yes)
@@
 			(project "ataconso-rev-a"
 				(path "/837c7b7b-d540-4609-998f-42c63488299f"
-					(reference "#PWR04")
+					(reference "#PWR09")
 					(unit 1)
 				)
@@
 		(in_pos_files yes)
 		(dnp no)
-		(property "Reference" "C4"
+		(property "Reference" "C3"
 			(at 85.09 71.1199 0)
 			(show_name no)
@@
 			(project "ataconso-rev-a"
 				(path "/837c7b7b-d540-4609-998f-42c63488299f"
-					(reference "C4")
+					(reference "C3")
 					(unit 1)
 				)
@@
 		(dnp no)
 		(fields_autoplaced yes)
-		(property "Reference" "#PWR06"
+		(property "Reference" "#PWR012"
 			(at 111.76 49.53 0)
 			(hide yes)
@@
 			(project "ataconso-rev-a"
 				(path "/837c7b7b-d540-4609-998f-42c63488299f"
-					(reference "#PWR06")
+					(reference "#PWR012")
+					(unit 1)
+				)
+			)
+		)
+	)
+	(symbol
+		(lib_id "Device:C")
+		(at 33.02 72.39 0)
+		(mirror y)
+		(unit 1)
+		(body_style 1)
+		(exclude_from_sim no)
+		(in_bom yes)
+		(on_board yes)
+		(in_pos_files yes)
+		(dnp no)
+		(property "Reference" "C1"
+			(at 29.21 71.1199 0)
+			(show_name no)
+			(do_not_autoplace no)
+			(effects
+				(font
+					(size 1.27 1.27)
+				)
+				(justify left)
+			)
+		)
+		(property "Value" "10n"
+			(at 29.21 73.6599 0)
+			(show_name no)
+			(do_not_autoplace no)
+			(effects
+				(font
+					(size 1.27 1.27)
+				)
+				(justify left)
+			)
+		)
+		(property "Footprint" ""
+			(at 32.0548 76.2 0)
+			(hide yes)
+			(show_name no)
+			(do_not_autoplace no)
+			(effects
+				(font
+					(size 1.27 1.27)
+				)
+			)
+		)
+		(property "Datasheet" ""
+			(at 33.02 72.39 0)
+			(hide yes)
+			(show_name no)
+			(do_not_autoplace no)
+			(effects
+				(font
+					(size 1.27 1.27)
+				)
+			)
+		)
+		(property "Description" "Unpolarized capacitor"
+			(at 33.02 72.39 0)
+			(hide yes)
+			(show_name no)
+			(do_not_autoplace no)
+			(effects
+				(font
+					(size 1.27 1.27)
+				)
+			)
+		)
+		(pin "1"
+		)
+		(pin "2"
+		)
+		(instances
+			(project "ataconso-rev-a"
+				(path "/837c7b7b-d540-4609-998f-42c63488299f"
+					(reference "C1")
 					(unit 1)
 				)
@@
 		(dnp no)
 		(fields_autoplaced yes)
-		(property "Reference" "#PWR09"
+		(property "Reference" "#PWR01"
 			(at 30.48 49.53 0)
 			(hide yes)
@@
 			(project "ataconso-rev-a"
 				(path "/837c7b7b-d540-4609-998f-42c63488299f"
-					(reference "#PWR09")
+					(reference "#PWR01")
 					(unit 1)
 				)
@@
 		(in_pos_files yes)
 		(dnp no)
-		(property "Reference" "C1"
+		(property "Reference" "C2"
 			(at 49.53 31.7499 0)
 			(show_name no)
@@
 			(project "ataconso-rev-a"
 				(path "/837c7b7b-d540-4609-998f-42c63488299f"
-					(reference "C1")
+					(reference "C2")
 					(unit 1)
 				)
@@
 		(dnp no)
 		(fields_autoplaced yes)
-		(property "Reference" "#PWR05"
+		(property "Reference" "#PWR06"
 			(at 60.96 49.53 0)
 			(hide yes)
@@
 			(project "ataconso-rev-a"
 				(path "/837c7b7b-d540-4609-998f-42c63488299f"
-					(reference "#PWR05")
+					(reference "#PWR06")
 					(unit 1)
 				)
@@
 		(dnp no)
 		(fields_autoplaced yes)
-		(property "Reference" "#PWR011"
+		(property "Reference" "#PWR07"
 			(at 88.9 83.82 0)
 			(hide yes)
@@
 			(project "ataconso-rev-a"
 				(path "/837c7b7b-d540-4609-998f-42c63488299f"
-					(reference "#PWR011")
+					(reference "#PWR07")
 					(unit 1)
 				)
@@
 	)
 	(symbol
-		(lib_id "Device:C_Polarized")
-		(at 33.02 72.39 0)
-		(unit 1)
-		(body_style 1)
-		(exclude_from_sim no)
-		(in_bom yes)
-		(on_board yes)
-		(in_pos_files yes)
-		(dnp no)
-		(fields_autoplaced yes)
-		(property "Reference" "C2"
-			(at 36.83 70.2309 0)
-			(show_name no)
-			(do_not_autoplace no)
-			(effects
-				(font
-					(size 1.27 1.27)
-				)
-				(justify left)
-			)
-		)
-		(property "Value" "10u"
-			(at 36.83 72.7709 0)
-			(show_name no)
-			(do_not_autoplace no)
-			(effects
-				(font
-					(size 1.27 1.27)
-				)
-				(justify left)
-			)
-		)
-		(property "Footprint" ""
-			(at 33.9852 76.2 0)
-			(hide yes)
-			(show_name no)
-			(do_not_autoplace no)
-			(effects
-				(font
-					(size 1.27 1.27)
-				)
-			)
-		)
-		(property "Datasheet" ""
-			(at 33.02 72.39 0)
-			(hide yes)
-			(show_name no)
-			(do_not_autoplace no)
-			(effects
-				(font
-					(size 1.27 1.27)
-				)
-			)
-		)
-		(property "Description" "Polarized capacitor"
-			(at 33.02 72.39 0)
-			(hide yes)
-			(show_name no)
-			(do_not_autoplace no)
-			(effects
-				(font
-					(size 1.27 1.27)
-				)
-			)
-		)
-		(pin "1"
-		)
-		(pin "2"
-		)
-		(instances
-			(project "ataconso-rev-a"
-				(path "/837c7b7b-d540-4609-998f-42c63488299f"
-					(reference "C2")
-					(unit 1)
-				)
-			)
-		)
-	)
-	(symbol
 		(lib_id "Timer:NE555D")
 		(at 58.42 58.42 0)
@@
 		(in_pos_files yes)
 		(dnp no)
-		(property "Reference" "C3"
+		(property "Reference" "C4"
 			(at 100.33 31.7499 0)
 			(show_name no)
@@
 			(project "ataconso-rev-a"
 				(path "/837c7b7b-d540-4609-998f-42c63488299f"
-					(reference "C3")
+					(reference "C4")
 					(unit 1)
 				)
@@
 		(dnp no)
 		(fields_autoplaced yes)
-		(property "Reference" "#PWR02"
+		(property "Reference" "#PWR011"
 			(at 109.22 83.82 0)
 			(hide yes)
@@
 			(project "ataconso-rev-a"
 				(path "/837c7b7b-d540-4609-998f-42c63488299f"
-					(reference "#PWR02")
+					(reference "#PWR011")
 					(unit 1)
 				)
@@
 		(dnp no)
 		(fields_autoplaced yes)
-		(property "Reference" "#PWR07"
+		(property "Reference" "#PWR04"
 			(at 53.34 45.72 0)
 			(hide yes)
@@
 			(project "ataconso-rev-a"
 				(path "/837c7b7b-d540-4609-998f-42c63488299f"
-					(reference "#PWR07")
+					(reference "#PWR04")
 					(unit 1)
 				)
@@
 		(dnp no)
 		(fields_autoplaced yes)
-		(property "Reference" "#PWR012"
+		(property "Reference" "#PWR08"
 			(at 92.71 27.94 0)
 			(hide yes)
@@
 			(project "ataconso-rev-a"
 				(path "/837c7b7b-d540-4609-998f-42c63488299f"
-					(reference "#PWR012")
-					(unit 1)
-				)
+					(reference "#PWR08")
+					(unit 1)
+				)

Commit message: cambiar valores de componentes
Parts:
- C3: value 100n -> 10n
- C5: value C_Polarized -> 100u
- R1: value 1k -> 10k
Other:
- note added: "555 izquierda 1: a tierra 2: a tierra por C 3: a 2 de 555 derecha 4: a Vcc 5: a tierra por C 6: a 2 7: a Vcc por R, a 2 por RV 8: a Vcc"
- note removed: "555 izquierda 1: a tierra 2: a tierra por C 3: a 2 de 555 derecha 4: a Vcc 5: a tierra por C 100n 6: a 2 7: a Vcc por R 10k, a 2 por RV de 100k 8: a Vcc"
Changed lines of the file:
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@@
 		)
 	)
-	(text "555 izquierda\n1: a tierra\n2: a tierra por C\n3: a 2 de 555 derecha\n4: a Vcc\n5: a tierra por C 100n\n6: a 2\n7: a Vcc por R 10k, a 2 por RV de 100k\n8: a Vcc"
+	(text "555 izquierda\n1: a tierra\n2: a tierra por C\n3: a 2 de 555 derecha\n4: a Vcc\n5: a tierra por C\n6: a 2\n7: a Vcc por R, a 2 por RV\n8: a Vcc"
 		(exclude_from_sim no)
 		(at 17.78 102.108 0)
@@
 			)
 		)
-		(property "Value" "100n"
+		(property "Value" "10n"
 			(at 85.09 73.6599 0)
 			(show_name no)
@@
 			)
 		)
-		(property "Value" "1k"
+		(property "Value" "10k"
 			(at 33.02 53.3399 0)
 			(show_name no)
@@
 			)
 		)
-		(property "Value" "C_Polarized"
+		(property "Value" "100u"
 			(at 137.541 53.34 90)
 			(show_name no)

Commit message: añadida alimentación y corregidos valores
Parts:
- added D1: 1n4007, symbol Device:D
- added D2: LED, symbol Device:LED
- added J2: Barrel_Jack_Switch, Connector_BarrelJack:BarrelJack_Horizontal, symbol Connector:Barrel_Jack_Switch
- added R3: 1k, symbol Device:R
- added SW1: SW_SPDT, symbol Switch:SW_SPDT
- C3: value 10n -> 100n
- RV1, RV2: value 100k -> 470k
Connections:
- net GND: now also J2.2, J2.3, R3.2
- net VCC: now also D1.1 (K), D2.2 (A)
- new net: J2.1, SW1.2 (B)
- new net: D2.1 (K), R3.1
- new net: D1.2 (A), SW1.3 (C)

Commit message: agregar pcb
Parts:
- C1, C2, C3, C4: footprint (none) -> Capacitor_THT:C_Disc_D3.8mm_W2.6mm_P2.50mm
- C5: footprint (none) -> Capacitor_THT:CP_Radial_D5.0mm_P2.50mm
- D1: footprint (none) -> Diode_THT:D_DO-41_SOD81_P10.16mm_Horizontal
- D2: footprint (none) -> LED_THT:LED_D5.0mm
- J1: footprint (none) -> TerminalBlock:TerminalBlock_MaiXu_MX126-5.0-02P_1x02_P5.00mm
- R1, R2, R3: footprint (none) -> Resistor_THT:R_Axial_DIN0207_L6.3mm_D2.5mm_P10.16mm_Horizontal
- RV1, RV2: footprint (none) -> Potentiometer_THT:Potentiometer_Piher_PT-6-V_Vertical
- SW1: footprint (none) -> parla:spdt_ssd12d00g3
Changed lines of the file:
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@@
 			)
 		)
-		(property "Footprint" ""
+		(property "Footprint" "Resistor_THT:R_Axial_DIN0207_L6.3mm_D2.5mm_P10.16mm_Horizontal"
 			(at 87.122 45.72 90)
 			(hide yes)
@@
 			)
 		)
-		(property "Footprint" ""
+		(property "Footprint" "Resistor_THT:R_Axial_DIN0207_L6.3mm_D2.5mm_P10.16mm_Horizontal"
 			(at 179.197 41.275 90)
 			(hide yes)
@@
 			)
 		)
-		(property "Footprint" ""
+		(property "Footprint" "Capacitor_THT:C_Disc_D3.8mm_W2.6mm_P2.50mm"
 			(at 87.9348 76.2 0)
 			(hide yes)
@@
 			)
 		)
-		(property "Footprint" ""
+		(property "Footprint" "Capacitor_THT:C_Disc_D3.8mm_W2.6mm_P2.50mm"
 			(at 32.0548 76.2 0)
 			(hide yes)
@@
 			)
 		)
-		(property "Footprint" ""
+		(property "Footprint" "Potentiometer_THT:Potentiometer_Piher_PT-6-V_Vertical"
 			(at 21.59 59.69 0)
 			(hide yes)
@@
 			)
 		)
-		(property "Footprint" ""
+		(property "Footprint" "parla:spdt_ssd12d00g3"
 			(at 161.925 21.59 0)
 			(hide yes)
@@
 			)
 		)
-		(property "Footprint" ""
+		(property "Footprint" "Resistor_THT:R_Axial_DIN0207_L6.3mm_D2.5mm_P10.16mm_Horizontal"
 			(at 28.702 52.07 90)
 			(hide yes)
@@
 			)
 		)
-		(property "Footprint" ""
+		(property "Footprint" "Capacitor_THT:C_Disc_D3.8mm_W2.6mm_P2.50mm"
 			(at 52.3748 36.83 0)
 			(hide yes)
@@
 			)
 		)
-		(property "Footprint" ""
+		(property "Footprint" "TerminalBlock:TerminalBlock_MaiXu_MX126-5.0-02P_1x02_P5.00mm"
 			(at 156.21 58.42 0)
 			(hide yes)
@@
 			)
 		)
-		(property "Footprint" ""
+		(property "Footprint" "Capacitor_THT:CP_Radial_D5.0mm_P2.50mm"
 			(at 142.24 57.4548 0)
 			(hide yes)
@@
 			)
 		)
-		(property "Footprint" ""
+		(property "Footprint" "Diode_THT:D_DO-41_SOD81_P10.16mm_Horizontal"
 			(at 173.99 24.13 0)
 			(hide yes)
@@
 			)
 		)
-		(property "Footprint" ""
+		(property "Footprint" "Capacitor_THT:C_Disc_D3.8mm_W2.6mm_P2.50mm"
 			(at 103.1748 36.83 0)
 			(hide yes)
@@
 			)
 		)
-		(property "Footprint" ""
+		(property "Footprint" "LED_THT:LED_D5.0mm"
 			(at 180.975 31.115 0)
 			(hide yes)
@@
 			)
 		)
-		(property "Footprint" ""
+		(property "Footprint" "Potentiometer_THT:Potentiometer_Piher_PT-6-V_Vertical"
 			(at 88.9 27.94 0)
 			(hide yes)

Commit message: agregar primera version
Parts:
- added H1, H2: MountingHole, MountingHole:MountingHole_3.2mm_M3, symbol Mechanical:MountingHole
Changed lines of the file:
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@@
+	)
+	(symbol
+		(lib_id "Mechanical:MountingHole")
+		(at 172.72 87.63 0)
+		(unit 1)
+		(body_style 1)
+		(exclude_from_sim no)
+		(in_bom no)
+		(on_board yes)
+		(in_pos_files yes)
+		(dnp no)
+		(fields_autoplaced yes)
+		(property "Reference" "H2"
+			(at 175.26 86.3599 0)
+			(show_name no)
+			(do_not_autoplace no)
+			(effects
+				(font
+					(size 1.27 1.27)
+				)
+				(justify left)
+			)
+		)
+		(property "Value" "MountingHole"
+			(at 175.26 88.8999 0)
+			(show_name no)
+			(do_not_autoplace no)
+			(effects
+				(font
+					(size 1.27 1.27)
+				)
+				(justify left)
+			)
+		)
+		(property "Footprint" "MountingHole:MountingHole_3.2mm_M3"
+			(at 172.72 87.63 0)
+			(hide yes)
+			(show_name no)
+			(do_not_autoplace no)
+			(effects
+				(font
+					(size 1.27 1.27)
+				)
+			)
+		)
+		(property "Datasheet" ""
+			(at 172.72 87.63 0)
+			(hide yes)
+			(show_name no)
+			(do_not_autoplace no)
+			(effects
+				(font
+					(size 1.27 1.27)
+				)
+			)
+		)
+		(property "Description" "Mounting Hole without connection"
+			(at 172.72 87.63 0)
+			(hide yes)
+			(show_name no)
+			(do_not_autoplace no)
+			(effects
+				(font
+					(size 1.27 1.27)
+				)
+			)
+		)
+		(instances
+			(project "ataconso-rev-a"
+				(path "/837c7b7b-d540-4609-998f-42c63488299f"
+					(reference "H2")
+					(unit 1)
+				)
+			)
+		)
 	)
 	(symbol
@@
 					(unit 1)
 				)
+			)
+		)
+	)
+	(symbol
+		(lib_id "Mechanical:MountingHole")
+		(at 149.86 87.63 0)
+		(unit 1)
+		(body_style 1)
+		(exclude_from_sim no)
+		(in_bom no)
+		(on_board yes)
+		(in_pos_files yes)
+		(dnp no)
+		(fields_autoplaced yes)
+		(property "Reference" "H1"
+			(at 152.4 86.3599 0)
+			(show_name no)
+			(do_not_autoplace no)
+			(effects
+				(font
+					(size 1.27 1.27)
+				)
+				(justify left)
+			)
+		)
+		(property "Value" "MountingHole"
+			(at 152.4 88.8999 0)
+			(show_name no)
+			(do_not_autoplace no)
+			(effects
+				(font
+					(size 1.27 1.27)
+				)
+				(justify left)
+			)
+		)
+		(property "Footprint" "MountingHole:MountingHole_3.2mm_M3"
+			(at 149.86 87.63 0)
+			(hide yes)
+			(show_name no)
+			(do_not_autoplace no)
+			(effects
+				(font
+					(size 1.27 1.27)
+				)
+			)
+		)
+		(property "Datasheet" ""
+			(at 149.86 87.63 0)
+			(hide yes)
+			(show_name no)
+			(do_not_autoplace no)
+			(effects
+				(font
+					(size 1.27 1.27)
+				)
+			)
+		)
+		(property "Description" "Mounting Hole without connection"
+			(at 149.86 87.63 0)
+			(hide yes)
+			(show_name no)
+			(do_not_autoplace no)
+			(effects
+				(font
+					(size 1.27 1.27)
+				)
+			)
+		)
+		(instances
+			(project "ataconso-rev-a"
+				(path "/837c7b7b-d540-4609-998f-42c63488299f"
+					(reference "H1")
+					(unit 1)
+				)
