File: ataconso/ataconso-rev-b/ataconso-rev-b.kicad_pcb (KiCad board)
At the start: 2 copper layers, 20 x 100 mm, 17 parts, among them J1 Screw_Terminal_01x02, J2 Barrel_Jack_Switch, SW1 SW_SPDT, U1 NE555D, U2 NE555D

Commit message: agregar pcb de rev-b
Parts:
- moved R2 11.2 mm to (53.0, 126.0), turned to -90 degrees
- moved C4 6.80 mm to (58.0, 127.0)
- moved C3 5.39 mm to (63.5, 131.0)
Routing:
- net VCC: track 0.00 -> 84.0 mm
- net Net-(U1-THRES): track 0.00 -> 69.4 mm
- net Net-(U2-DISCH): track 0.00 -> 50.9 mm
- net Net-(D1-A): track 0.00 -> 49.8 mm
- net Net-(U2-OUT): track 0.00 -> 41.3 mm
- net Net-(U1-DISCH): track 0.00 -> 36.9 mm
- net Net-(U2-CONT): track 0.00 -> 22.0 mm
- net Net-(U1-CONT): track 0.00 -> 21.7 mm
- net Net-(R2-Pad1): track 0.00 -> 17.8 mm
- net Net-(U1-OUT): track 0.00 -> 14.4 mm
- net Net-(SW1-B): track 0.00 -> 13.5 mm
- net Net-(D2-K): track 0.00 -> 13.3 mm
- net Net-(J1-Pin_1): track 0.00 -> 12.2 mm
Other:
- board text added: "ataconso"
- board text added: "rev-b 08-2026"

Commit message: agregar avances rev-b
Parts:
- moved D2 2.00 mm to (63.7, 66.0)
- moved J2 1.00 mm to (57.0, 65.0)
Routing:
- net Net-(D1-A): track 49.8 -> 53.5 mm
- net Net-(SW1-B): track 13.5 -> 15.4 mm
- net Net-(U2-DISCH): track 50.9 -> 49.2 mm
- added copper zone on B.Cu, net GND
- added copper zone on F.Cu, net GND
